Commit message: gui is working with vision and apple selection working. have tested on apples on a table but not on proxy or real wall of apples

File: harvest_control/resource/urdf/v_trellis_template.xacro (robot description, xacro)
@@ -1,7 +1,16 @@
 <?xml version="1.0"?>
+<!--
+  Simple V-trellis tree template (environment model, not part of the robot):
+  one vertical leader branch plus 4 horizontal branches spaced evenly up it.
+  UNITS: meters and radians.
+  v_trellis_template.urdf next to this file is GENERATED from it. After editing, regenerate:
+    xacro v_trellis_template.xacro -o v_trellis_template.urdf
+-->
 <robot name="tree_structure" xmlns:xacro="http://www.ros.org/wiki/xacro">
   <!-- Parameters for branches -->
   <xacro:property name="horizontal_branch_spacing" value="1.0"/> <!-- Spacing between horizontal branches -->
-  <xacro:property name="branch_diameter" value="0.04"/>          <!-- Diameter of the horizontal branches -->
+  <!-- NOTE: despite the name, branch_diameter is used as the cylinder RADIUS below,
+       so 0.04 gives 8 cm thick branches. -->
+  <xacro:property name="branch_diameter" value="0.04"/>          <!-- Radius of the horizontal branches (see note) -->
   <xacro:property name="branch_length" value="4.0"/>              <!-- Length of the horizontal branches -->
   <xacro:property name="leader_branch_radius" value="0.08"/>      <!-- Radius of the leader branch -->

File: harvest_hardware/robot_custom_hardware/urdf/_d435i.urdf.xacro (robot description, xacro)
@@ -18,4 +18,13 @@
 This is the URDF model for the Intel RealSense 435i camera, in it's
 aluminum peripherial evaluation case.
+LOCAL COPY of realsense2_description's _d435i.urdf.xacro, changed to take a "prefix" param so
+the robot can have two cameras (mast_camera_*, base_camera_*) without frame-name clashes.
+amiga_ur_gripper.urdf.xacro includes this copy; ur_gripper.urdf.xacro uses the upstream one.
+Usage:
+  <xacro:sensor_d435i parent="some_link" prefix="mast_" use_nominal_extrinsics="true">
+    <origin xyz="..." rpy="..."/>   <- pose of the camera's bottom screw hole in parent
+  </xacro:sensor_d435i>
+Frames created: ${prefix}camera_bottom_screw_frame, ${prefix}camera_link, and (when
+use_nominal_extrinsics is true) ${prefix}camera_color_optical_frame, _depth_optical_frame, etc.
 -->
 <robot name="sensor_d435i" xmlns:xacro="http://ros.org/wiki/xacro">

File: harvest_hardware/robot_custom_hardware/urdf/amiga.urdf.xacro (robot description, xacro)
@@ -1,3 +1,16 @@
 <?xml version="1.0"?>
+<!--
+  Amiga platform with the arm-mount frame on top.
+  Links (all named with amiga_prefix, default "amiga__"):
+    base   root of the Amiga, attached to amiga_parent (world) with no offset
+    body   the frame mesh plus collision boxes for the things bolted to it
+    tool0  where the UR5e base mounts (the arm's base_link is attached here)
+  All positions are relative to amiga__base / amiga__body (the same frame).
+  UNITS: meters and radians. Several values are inch measurements converted to m
+  (e.g. 1.04775 m = 41.25 in, 0.29845 m = 11.75 in).
+  Used by amiga_ur_gripper.urdf.xacro.
+  Keep a small gap between these boxes and the UR5e (e.g. the rail top is at z 1.045,
+  2.75 mm under the arm base at 1.04775). Touching boxes read as a self-collision in MoveIt.
+-->
 <robot xmlns:xacro="https://ros.org/wiki/xacro" name="amiga">
 <xacro:macro name="amiga_macro" params="amiga_prefix:='amiga__' amiga_parent:='world' mesh_base_path">
@@ -8,4 +21,6 @@
         <color rgba="0.941 0.941 0.941 1.0"/>
     </material>
+    <!-- Mass and overall box (box0) are used only for the inertia estimate below.
+         box1 / box2 are currently unused. -->
     <xacro:property name="amiga_mass" value="40.0"/>
     <xacro:property name="amiga_collision_box0_x" value='1.132'/>
@@ -18,4 +33,8 @@
     <xacro:property name="amiga_collision_box2_y" value='0.25' />
     <xacro:property name="amiga_collision_box2_z" value='0.25' />
+    <!-- ARM MOUNT: pose of the UR5e base on the Amiga, relative to amiga__body.
+         position: x -0.095, y 0.306, z 1.04775 (41.25 in up, sitting on top of the rail)
+         rotation: arm base yawed 45 deg (pi/4)
+         Moving the arm on the Amiga = change these two values. -->
     <xacro:property name="amiga_tool0_mount_rotation" value="0.0 0.0 ${pi / 4}"/>
     <xacro:property name="amiga_tool0_mount_position" value="-0.095 0.306 1.04775"/>
@@ -24,5 +43,9 @@
     <!-- ================== -->
     <link name="${amiga_prefix}base"/>
+    <!-- Each part below is an <origin> (box CENTER, relative to the body) plus a <box size>
+         (full x y z lengths). Every box appears twice, once as collision (what MoveIt avoids)
+         and once as visual (what RViz shows); keep the two in sync. -->
     <link name="${amiga_prefix}body">
+        <!-- Amiga frame mesh (visual) -->
         <visual>
             <origin rpy="0.0 0.0 0.0" xyz="0.0 0.0 0.0"/>
@@ -32,5 +55,6 @@
             <material name="LightLightGrey"/>
         </visual>
-        <!-- Linear Rail -->
+        <!-- Linear Rail: 1.2 m long along x, centered 11.75 in (0.29845 m) toward +y,
+             top face at z 0.97 + 0.15/2 = 1.045 -->
         <collision>
             <origin rpy="0.0 0.0 0.0" xyz="0.0 0.29845 0.97"/>
@@ -45,5 +69,5 @@
             </geometry>
         </visual>
-        <!-- Mast -->
+        <!-- Mast: 7 x 7 cm upright post, 0.95 m tall, centered at z 1.03 -->
         <collision>
             <origin rpy="0.0 0.0 0.0" xyz="0.57 -0.15 1.03"/>
@@ -58,5 +82,5 @@
             </geometry>
         </visual>
-        <!-- GPS & Oak cameras -->
+        <!-- GPS & Oak cameras: box on top of the mast -->
         <collision>
             <origin rpy="0.0 0.0 0.0" xyz="0.57 -0.15 1.6"/>
@@ -71,5 +95,5 @@
             </geometry>
         </visual>
-        <!-- Amiga Brain -->
+        <!-- Amiga Brain: box on the side of the mast -->
         <collision>
             <origin rpy="0.0 0.0 0.0" xyz="0.57 -0.315 1.25"/>
@@ -84,5 +108,5 @@
             </geometry>
         </visual>
-        <!-- Base -->
+        <!-- Base: the frame mesh as a collision shape -->
         <collision>
             <origin rpy="0.0 0.0 0.0" xyz="0.0 0.0 0.0"/>
@@ -91,4 +115,5 @@
             </geometry>
         </collision>
+        <!-- Rough inertia: 40 kg solid box of size box0. Only matters for simulation. -->
         <inertial>
             <origin rpy="0 0 0" xyz="0.0 0.0 0.0"/>
@@ -103,4 +128,5 @@
         </inertial>
     </link>
+    <!-- Arm mount frame; the UR5e base_link attaches here -->
     <link name="${amiga_prefix}tool0"/>
     <!-- ================== -->
@@ -117,4 +143,5 @@
         <child link="${amiga_prefix}body"/>
     </joint>
+    <!-- Arm mount pose; values come from the ARM MOUNT properties at the top -->
     <joint name="${amiga_prefix}body--${amiga_prefix}tool0" type="fixed">
         <origin rpy="${amiga_tool0_mount_rotation}" xyz="${amiga_tool0_mount_position}"/>

File: harvest_hardware/robot_custom_hardware/urdf/amiga_ur_gripper.urdf.xacro (robot description, xacro)
@@ -1,5 +1,25 @@
 <?xml version="1.0"?>
+<!--
+  FULL ROBOT: Amiga platform + UR5e arm + gripper/ejector + two RealSense D435i cameras.
+  Tree:  world -> amiga__base -> amiga__body -> amiga__tool0 (arm mount)
+           -> UR5e (base_link ... wrist_3_link -> flange -> tool0)
+                tool0 -> gripper_link (tip), ejector_link, mast camera, tracking marker
+         amiga__base -> base camera
+  Pieces live in:
+    amiga.urdf.xacro    Amiga frame, its collision boxes, and where the arm mounts
+    gripper.urdf.xacro  gripper body, ejector, suction-cup / palm / top camera frames
+    _d435i.urdf.xacro   local copy of the RealSense macro with a "prefix" param added
+  The arm + gripper WITHOUT the Amiga is ur_gripper.urdf.xacro. It duplicates gripper_joint
+  below; keep the two in sync.
+  UNITS: meters and radians (inches x 0.0254 = m, degrees x pi/180 = rad).
+  tool0 axes: +z out of the flange along the gripper, -y toward the ejector/mast-camera side.
+  To build by hand (e.g. to check a change):
+    xacro amiga_ur_gripper.urdf.xacro name:=ur -o /tmp/robot.urdf && check_urdf /tmp/robot.urdf
+  (name:=ur is needed because <robot name> is read before the default below is declared.)
+  Restart robot_state_publisher / MoveIt / RViz to pick up changes; no rebuild needed
+  (install/ symlinks back to these files).
+-->
 <robot xmlns:xacro="http://www.ros.org/wiki/xacro" name="$(arg name)">
-  <!-- keep the basics -->
+  <!-- UR driver args: these just pass through to ur_robot below. Launch files set most of them. -->
   <xacro:arg name="name" default="ur"/>
   <xacro:arg name="ur_type" default="ur5e"/>  <!-- absorbs CLI arg; we won't pass it to ur_robot -->
@@ -33,9 +53,13 @@
   <xacro:arg name="sim_ignition" default="false"/>
   <xacro:arg name="simulation_controllers" default=""/>
+  <!-- Joint angles the arm starts at in fake hardware / simulation -->
   <xacro:arg name="initial_positions_file" default="$(find robot_custom_hardware)/config/initial_positions.yaml"/>
   <xacro:property name="initial_positions_file" default="$(arg initial_positions_file)"/>
-  <!-- Amiga args -->
+  <!-- Amiga args: prefix for every Amiga link name (amiga__base, amiga__body, amiga__tool0) -->
   <xacro:arg name="amiga_prefix" default="amiga__"/>
-  <!-- Realsense args -->
+  <!-- Realsense args.
+       true:  the URDF includes each camera's internal frames (depth / color / infra optical)
+              at nominal factory offsets, e.g. mast_camera_color_optical_frame.
+       false: the realsense driver must publish those frames itself. -->
   <xacro:arg name="use_nominal_extrinsics" default="true" />
   <!-- Define the four args with the names the UR macro expects -->
@@ -55,5 +79,5 @@
   <xacro:property name="robot_custom_hardware" value="package://robot_custom_hardware/"/>
   <xacro:amiga_macro amiga_prefix="$(arg amiga_prefix)" amiga_parent="world" mesh_base_path="package://robot_custom_hardware/meshes/"/>
-  <!-- UR5e arm -->
+  <!-- UR5e arm, mounted on amiga__tool0 (mount pose is set in amiga.urdf.xacro) -->
   <xacro:ur_robot
       name="$(arg name)"
@@ -94,19 +118,34 @@
     <origin xyz="0 0 0" rpy="0 0 0"/>
   </xacro:ur_robot>
-  <!-- mount gripper -->
+  <!-- Gripper mount: gripper_link = the gripper TIP, 25 cm straight out from the flange
+       (the gripper spans 1-25 cm). MoveIt drives this frame to pick targets, and
+       start_harvest.py trigger_move_arm_to_pose stops it 15 cm short (world -y) of the apple.
+       If you change this z:
+         - make the same change in ur_gripper.urdf.xacro
+         - shift the frames in gripper.urdf.xacro (they're relative to the tip)
+         - recompute the gripper box center in gripper.urdf.xacro -->
   <joint name="gripper_joint" type="fixed">
     <parent link="tool0"/>
     <child  link="gripper_link"/>
-    <origin xyz="0.00 0.00 0.215" rpy="0 0 0"/>
+    <origin xyz="0.00 0.00 0.25" rpy="0 0 0"/>
   </joint>
+  <!-- Gripper body, ejector plate, suction-cup / palm / top camera frames -->
   <xacro:gripper_macro/>
-  <!-- MAST Realsense for apple locations -->
+  <!-- MAST RealSense (on the wrist), used for apple locations; apple_prediction.py reads
+       mast_camera_color_optical_frame.
+       Origin = the camera's bottom screw hole, relative to tool0:
+         y = -0.09   9 cm over the wrist center (ejector side)
+         z = 0.055   5.5 cm out from the flange
+       rpy: the camera looks along +z (same direction as the gripper) with its top facing -y
+       (away from the wrist). If apple positions come out mirrored or flipped, check this rotation. -->
   <xacro:sensor_d435i
     parent="tool0"
     prefix="mast_"
     use_nominal_extrinsics="$(arg use_nominal_extrinsics)">
-    <origin xyz="0.0 0.09 0.05" rpy="0 -1.57 -1.57"/>
+    <origin xyz="0.0 -0.09 0.055" rpy="0 -1.57 1.57"/>
   </xacro:sensor_d435i>
-  <!-- Realsense for trunk detections -->
+  <!-- BASE RealSense (fixed on the Amiga), used for trunk detections.
+       Relative to amiga__base: 0.3937 m (15.5 in) along +y, 0.5556 m (21.875 in) up,
+       yawed 90 deg. -->
   <xacro:sensor_d435i
     parent="$(arg amiga_prefix)base"
@@ -115,5 +154,7 @@
     <origin xyz="0.0 0.3937 0.555625" rpy="0 0 1.57"/>
   </xacro:sensor_d435i>
-  <!-- Tracking marker frame -->
+  <!-- Tracking marker frame on the tool: 12 cm toward +y (the side opposite the ejector),
+       3.7 cm out from the flange. Frame only; the 1 mm red sphere just makes it visible in
+       RViz. No code references it by name. If the physical marker moved, update this. -->
   <joint name="tracking_marker_joint" type="fixed">
     <parent link="tool0"/>

File: harvest_hardware/robot_custom_hardware/urdf/gripper.urdf.xacro (robot description, xacro)
@@ -1,11 +1,33 @@
 <?xml version="1.0"?>
+<!--
+  End-of-arm tooling: gripper body, ejector plate, and the gripper's reference frames.
+  Used by both amiga_ur_gripper.urdf.xacro and ur_gripper.urdf.xacro. Those files create
+  gripper_joint (tool0 -> gripper_link); this macro builds everything hanging off it.
+  UNITS: meters and radians (inches x 0.0254 = m, degrees x pi/180 = rad).
+  tool0 FRAME (the UR flange, where everything here is measured from):
+    origin = center of the flange face
+    +z     = straight out of the flange, along the gripper
+    -y     = the side the ejector and mast camera are on ("over" the wrist)
+    +y     = the opposite side ("under" the wrist)
+  The wrist_3 body behind the flange is a cylinder of radius ~3.75 cm (UR5e collision mesh).
+-->
 <robot xmlns:xacro="http://www.ros.org/wiki/xacro">
     <xacro:macro name="gripper_macro">
+        <!-- ============================================================ -->
+        <!--  Frames on the gripper (offsets are from gripper_link, the   -->
+        <!--  tip, so negative z = back toward the flange).               -->
+        <!--  If you change gripper_joint's z in the top-level files,     -->
+        <!--  change these z values by the opposite amount to keep the    -->
+        <!--  frames where they physically are.                           -->
+        <!-- ============================================================ -->
+        <!-- Suction cups: 19.5 cm from the flange (0.25 - 0.055).
+             Yaw of -150 deg lines the frame up with the cup pattern. -->
         <joint name="gripper_scups_joint" type="fixed">
             <parent link="gripper_link" />
             <child link="gripper_scups_link" />
-            <origin xyz="0.00 0.00 -0.02" rpy="0 0 -2.618" />
+            <origin xyz="0.00 0.00 -0.055" rpy="0 0 -2.618" />
         </joint>
         <link name="gripper_scups_link">
+            <!-- Uncomment to see the frame as a small green cube in RViz -->
             <!-- <visual>
                 <geometry>
@@ -17,17 +39,21 @@
             </visual> -->
         </link>
+        <!-- Palm camera optical frame: 16.5 cm from the flange (0.25 - 0.085), on the tool axis.
+             gripper_palm_camera.py stamps its images with this frame; visual_servo.py uses it. -->
         <joint name="gripper_palm_camera_joint" type="fixed">
             <parent link="gripper_link" />
             <child link="gripper_palm_camera_optical_link" />
-            <origin xyz="0.00 0 -0.05" rpy="0 0 0" />
+            <origin xyz="0.00 0 -0.085" rpy="0 0 0" />
         </joint>
+        <!-- Top camera: 12.85 cm from the flange (0.25 - 0.1215), 7.2 cm toward -y (the ejector side). -->
         <joint name="gripper_top_camera_joint" type="fixed">
             <parent link="gripper_link" />
             <child link="gripper_top_camera_link" />
-            <origin xyz="0.00 -.072 -0.0865" rpy="0 0 0" />
+            <origin xyz="0.00 -.072 -0.1215" rpy="0 0 0" />
         </joint>
         <link name="gripper_top_camera_link">
         </link>
         <link name="gripper_palm_camera_optical_link">
+            <!-- Uncomment to see the frame as a small green box in RViz -->
             <!-- <visual>
                 <geometry>
@@ -39,16 +65,64 @@
             </visual> -->
         </link>
-        <link name="gripper_link">
+        <!-- ============================================================ -->
+        <!--  Ejector plate (measured on the robot)                       -->
+        <!--    22 cm wide (x) x 14 cm tall (y) x 2.5 cm thick (z)        -->
+        <!--    flush against the flange: z 0 to 0.025                   -->
+        <!--    bottom edge 1 cm above the wrist surface (3.75 + 1 cm),   -->
+        <!--    on the -y side: y -0.0475 to -0.1875                      -->
+        <!--  The joint origin is the plate's center:                     -->
+        <!--    y = -(0.0475 + 0.14/2) = -0.1175,  z = 0.025/2 = 0.0125   -->
+        <!--  If you resize it, update the box size AND the center.       -->
+        <!--  Clearance: ~1.25 cm to the gripper body, ~1.4 cm to the     -->
+        <!--  wrist. Keep a gap; if boxes overlap, MoveIt sees a          -->
+        <!--  permanent self-collision and refuses to plan.               -->
+        <!-- ============================================================ -->
+        <joint name="ejector_joint" type="fixed">
+            <parent link="tool0" />
+            <child link="ejector_link" />
+            <origin xyz="0 -0.1175 0.0125" rpy="0 0 0" />
+        </joint>
+        <link name="ejector_link">
         <collision>
-            <origin xyz="0 0 0" rpy="0 0 0" />
             <geometry>
-            <cylinder radius="0.05" length="0.285" />
+            <box size="0.22 0.14 0.025" />
             </geometry>
         </collision>
         <visual>
-            <origin xyz="0 0 0" rpy="0 0 0" />
             <geometry>
-            <cylinder radius="0.05" length="0.285" />
+            <box size="0.22 0.14 0.025" />
             </geometry>
+            <material name="gripper_aluminum">  <!-- same as the RealSense "aluminum" -->
+                <color rgba="0.5 0.5 0.5 1" />
+            </material>
+        </visual>
+        </link>
+        <!-- ============================================================ -->
+        <!--  Gripper body (measured on the robot)                        -->
+        <!--    square prism, 7 x 7 cm cross-section, 24 cm long          -->
+        <!--    starts 1 cm out from the flange, so it spans z 0.01-0.25  -->
+        <!--  gripper_link sits at the TIP (0.25, set by gripper_joint in -->
+        <!--  the top-level files). It is the frame MoveIt moves to the   -->
+        <!--  target (move_arm.cpp setPoseTarget) and the "gripper tip"   -->
+        <!--  in pose_listener.py / orchard_templating.py.                -->
+        <!--  The box center is 0.12 behind the tip:                      -->
+        <!--    0.25 - (0.01 + 0.24/2) = 0.12                             -->
+        <!--  If you change the length or start offset, recompute this.   -->
+        <!-- ============================================================ -->
+        <link name="gripper_link">
+        <collision>
+            <origin xyz="0 0 -0.12" rpy="0 0 0" />
+            <geometry>
+            <box size="0.07 0.07 0.24" />
+            </geometry>
+        </collision>
+        <visual>
+            <origin xyz="0 0 -0.12" rpy="0 0 0" />
+            <geometry>
+            <box size="0.07 0.07 0.24" />
+            </geometry>
+            <material name="gripper_aluminum">  <!-- same as the RealSense "aluminum" -->
+                <color rgba="0.5 0.5 0.5 1" />
+            </material>
         </visual>
         </link>

File: harvest_hardware/robot_custom_hardware/urdf/ur_gripper.urdf.xacro (robot description, xacro)
@@ -1,5 +1,18 @@
 <?xml version="1.0"?>
+<!--
+  ARM ONLY (no Amiga): UR5e fixed to world + gripper/ejector + one RealSense D435i on the arm base.
+  The full robot on the Amiga is amiga_ur_gripper.urdf.xacro.
+  Tree:  world -> UR5e (base_link ... tool0)
+           tool0 -> gripper_link (tip), ejector_link   (from gripper.urdf.xacro)
+           base_link -> camera
+  This file duplicates gripper_joint from amiga_ur_gripper.urdf.xacro; keep the two in sync.
+  Unlike the Amiga file it has no mast camera or tracking marker, and it uses the upstream
+  realsense2_description macro (no prefix param), so the camera frames are plain camera_*.
+  UNITS: meters and radians (inches x 0.0254 = m, degrees x pi/180 = rad).
+  To build by hand:
+    xacro ur_gripper.urdf.xacro name:=ur -o /tmp/robot.urdf && check_urdf /tmp/robot.urdf
+-->
 <robot xmlns:xacro="http://www.ros.org/wiki/xacro" name="$(arg name)">
-  <!-- keep the basics -->
+  <!-- UR driver args: these just pass through to ur_robot below. Launch files set most of them. -->
   <xacro:arg name="name" default="ur"/>
   <xacro:arg name="ur_type" default="ur5e"/>  <!-- absorbs CLI arg; we won't pass it to ur_robot -->
@@ -36,5 +49,8 @@
   <xacro:arg name="initial_positions_file" default="$(find robot_custom_hardware)/config/initial_positions.yaml"/>
   <xacro:property name="initial_positions_file" default="$(arg initial_positions_file)"/>
-  <!-- Realsense args -->
+  <!-- Realsense args.
+       true:  the URDF includes the camera's internal frames (depth / color / infra optical)
+              at nominal factory offsets.
+       false: (default here) the realsense driver must publish those frames itself. -->
   <xacro:arg name="use_nominal_extrinsics" default="false" />
   <!-- CRITICAL: define the four args with the names the UR macro expects -->
@@ -88,11 +104,16 @@
     <origin xyz="0 0 0" rpy="0 0 0"/>
   </xacro:ur_robot>
-  <!-- mount gripper -->
+  <!-- Gripper mount: gripper_link = the gripper TIP, 25 cm straight out from the flange.
+       MUST MATCH gripper_joint in amiga_ur_gripper.urdf.xacro; see the notes there on
+       what else to update when this changes. -->
   <joint name="gripper_joint" type="fixed">
     <parent link="tool0"/>
     <child  link="gripper_link"/>
-    <origin xyz="0.00 0.00 0.215" rpy="0 0 0"/>
+    <origin xyz="0.00 0.00 0.25" rpy="0 0 0"/>
   </joint>
+  <!-- Gripper body, ejector plate, suction-cup / palm / top camera frames -->
   <xacro:gripper_macro/>
+  <!-- RealSense fixed near the arm, relative to base_link: 0.476 m (18.75 in) x,
+       -0.491 m y, 0.467 m up, yawed 1.8852 rad (~108 deg). -->
   <xacro:sensor_d435i parent="base_link" use_nominal_extrinsics="$(arg use_nominal_extrinsics)">
     <origin xyz="0.47625 -0.4907 0.4667" rpy="0 0 1.8852"/>
